File: NANOFC.kicad_pcb (KiCad board)
At the start: 2 copper layers, 50 x 60 mm, 21 parts, among them J1 Power in, J10 P2 Arm, J11 Micro_SD_Card, J2 Pyro 1, J3 BMP 280, J4 Pyro 2, J5 SIG, J6 V+, J7 GND, J8 Master Arm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

Commit message: Fix
Fixed:
pyro channels
Added:
status leds
continuity test leds
breakers
Parts:
- added C2: 100nF, Capacitor_SMD:C_1210_3225Metric, B.Cu at (191.8, 83.5)
- added D2: Con2, LED_SMD:LED_PLCC-2, F.Cu at (164.9, 80.1)
- added D3: Con1, LED_SMD:LED_PLCC-2, F.Cu at (164.9, 71.1)
- added D4: LED, LED_SMD:LED_PLCC-2, F.Cu at (152.2, 111.5)
- added F1: Fuse, Fuse:Fuse_1206_3216Metric, B.Cu at (158.0, 71.1)
- added F2: Fuse, Fuse:Fuse_1206_3216Metric, B.Cu at (158.1, 80.2)
- added F3: Fuse, Fuse:Fuse_1206_3216Metric, B.Cu at (157.4, 111.9)
- added J12: UART, Connector_JST:JST_EH_B4B-EH-A_1x04_P2.50mm_Vertical, F.Cu at (167.6, 63.1)
- added JP1: SolderJumper_2_Open, Jumper:SolderJumper-2_P1.3mm_Open_Pad1.0x1.5mm, B.Cu at (158.0, 66.7)
- added JP2: SolderJumper_2_Open, Jumper:SolderJumper-2_P1.3mm_Open_Pad1.0x1.5mm, B.Cu at (158.1, 76.0)
- added JP3: SolderJumper_2_Open, Jumper:SolderJumper-2_P1.3mm_Open_Pad1.0x1.5mm, F.Cu at (169.8, 115.2)
- added R10: 300, Resistor_SMD:R_1210_3225Metric, B.Cu at (172.4, 63.8)
- added R11: 300, Resistor_SMD:R_1210_3225Metric, B.Cu at (169.1, 76.1)
- added R3: 100k, Resistor_SMD:R_1210_3225Metric, B.Cu at (176.5, 69.9)
- added R4: 100k, Resistor_SMD:R_1210_3225Metric, B.Cu at (179.7, 69.9)
- added R5: 100k, Resistor_SMD:R_1210_3225Metric, B.Cu at (182.9, 69.9)
- added R6: 100k, Resistor_SMD:R_1210_3225Metric, B.Cu at (186.2, 69.9)
- added R7: 100k, Resistor_SMD:R_1210_3225Metric, B.Cu at (189.4, 69.9)
- added R8: 65, LED_SMD:LED_1210_3225Metric, B.Cu at (152.2, 111.4)
- added R9: 100k, Resistor_SMD:R_1210_3225Metric, B.Cu at (168.9, 96.6)
- added U3: LTV-817S, Package_DIP:SMDIP-4_W9.53mm, B.Cu at (156.3, 86.8)
- added U4: W25Q128JVS, KP-PTR_lib:SON127P500X600X80-9N, B.Cu at (164.1, 99.6)
- BZ1, D1: moved to B.Cu
- J11: moved to F.Cu
- moved J9 34.7 mm to (161.3, 72.4)
- moved BZ1 34.5 mm to (155.4, 97.3), turned to 0 degrees
- moved J2 32.5 mm to (154.3, 72.9), turned to 90 degrees
- moved C1 32.3 mm to (178.0, 117.2), turned to -90 degrees
- moved J11 30.7 mm to (187.8, 81.0), turned to -90 degrees
- moved Q1 24.7 mm to (168.5, 70.2), turned to 180 degrees
- moved R1 21.9 mm to (164.5, 76.1), turned to 90 degrees
- moved J5 16.7 mm to (192.0, 111.4)
- moved J6 16.7 mm to (192.0, 114.2)
- moved J7 16.7 mm to (192.0, 117.0)
- moved J4 16.0 mm to (154.3, 81.9), turned to 90 degrees
- moved U1 14.6 mm to (172.7, 115.1)
- moved J8 14.5 mm to (166.7, 114.0)
- moved U2 12.2 mm to (180.1, 80.0), turned to 180 degrees
- moved Q2 11.2 mm to (168.5, 81.9)
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Connections:
- A1 pad 1: unconnected-(A1-Pad1) -> TX
- A1 pad 13: unconnected-(A1-Pad13) -> SPI_CS_FLASH
- A1 pad 2: unconnected-(A1-Pad2) -> RX
- A1 pad 7: Buzzer -> BuzzerPin
- BZ1 pad 1: Buzzer -> Net-(BZ1-Pad1)
- D1 pad 2: Net-(J1-Pad2) -> Net-(D1-Pad2)
- J1 pad 2: Net-(J1-Pad2) -> Net-(F3-Pad1)
- J10 pad 2: Net-(J10-Pad2) -> Net-(F2-Pad2)
- J11 pad 1: unconnected-(J11-Pad1) -> Net-(J11-Pad1)
- J11 pad 4: 3.3v -> Net-(C2-Pad1)
- J11 pad 8: unconnected-(J11-Pad8) -> Net-(J11-Pad8)
- J2 pad 2: Net-(J2-Pad2) -> Net-(F1-Pad1)
- J4 pad 2: Net-(J10-Pad2) -> Net-(F2-Pad1)
- J8 pad 2: Net-(J1-Pad2) -> Net-(F3-Pad1)
- J9 pad 2: Net-(J2-Pad2) -> Net-(F1-Pad2)
- U2 pad 6: Net-(J2-Pad1) -> +BATT
- U2 pad 8: Net-(J4-Pad1) -> +BATT
Routing:
- net GND: track 142.9 -> 21.7 mm, vias 0 -> 3
- net 3.3v: track 101.2 -> 200.5 mm, vias 0 -> 8
- net TX: track 0.00 -> 73.1 mm, vias 0 -> 3
- net RX: track 0.00 -> 71.6 mm, vias 0 -> 2
- net MOSI: track 21.0 -> 82.8 mm, vias 0 -> 5
- net CS: track 7.09 -> 52.8 mm, vias 0 -> 2
- net MISO: track 32.1 -> 75.7 mm, vias 0 -> 2
- net Buzzer: track 43.4 -> 0.00 mm
- net +BATT: track 119.6 -> 161.0 mm, vias 0 -> 6
- net BuzzerPin: track 0.00 -> 39.0 mm, vias 0 -> 4
- net SCK: track 83.1 -> 44.9 mm, vias 0 -> 2
- net SPI_CS_FLASH: track 0.00 -> 27.8 mm, vias 0 -> 2
- net Net-(C2-Pad1): track 0.00 -> 22.5 mm, vias 0 -> 1
- net Net-(Q2-Pad1): track 25.9 -> 4.01 mm
- net Net-(R10-Pad2): track 0.00 -> 18.8 mm, vias 0 -> 1
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- added copper zone on B.Cu, net GND
Other:
- board text added: "S1"
- board text added: "S2"
- board text added: "S3"
- board text added: "S4"
