File: NANOFC.kicad_sch (KiCad schematic)
At the start: 21 parts, among them J1 Power in, J10 P2 Arm, J11 Micro_SD_Card, J2 Pyro 1, J3 BMP 280, J4 Pyro 2, J5 SIG, J6 V+, J7 GND, J8 Master Arm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

Commit message: Fix
Fixed:
pyro channels
Added:
status leds
continuity test leds
breakers
Parts:
- added C2: 100nF, Capacitor_SMD:C_1210_3225Metric, symbol Device:C
- added D2, D3, D4: LED, LED_SMD:LED_PLCC-2, symbol Device:LED
- added F1, F2, F3: Fuse, Fuse:Fuse_1206_3216Metric, symbol Device:Fuse
- added J12: UART, Connector_JST:JST_EH_B4B-EH-A_1x04_P2.50mm_Vertical, symbol Connector:Conn_01x04_Male
- added JP1, JP2, JP3: SolderJumper_2_Open, Jumper:SolderJumper-2_P1.3mm_Open_Pad1.0x1.5mm, symbol Jumper:SolderJumper_2_Open
- added R10, R11: 300, Resistor_SMD:R_1210_3225Metric, symbol Device:R
- added R3, R4, R5, R6, R7, R9: 100k, Resistor_SMD:R_1210_3225Metric, symbol Device:R
- added R8: 65, LED_SMD:LED_1210_3225Metric, symbol Device:R
- added U3: LTV-817S, Package_DIP:SMDIP-4_W9.53mm, symbol Isolator:LTV-817S
- added U4: W25Q128JVS, KP-PTR_lib:SON127P500X600X80-9N, symbol Memory_Flash:W25Q128JVS
Connections:
- net +BATT: now also U2.6, U2.8, JP1.2 (B), JP2.2 (B), JP3.2 (B), U3.4
- net 3.3v: now also J12.3 (Pin_3), R3.2, R4.2, R5.2, R6.2, R7.2, R8.2, R9.1, U4.3 (IO2), U4.7 (IO3), U4.8 (VCC); no longer J11.4 (VDD)
- net CS: now also R4.1
- net GND: now also C2.2, D2.1 (K), D3.1 (K), D4.1 (K), J12.4 (Pin_4), U3.2, U4.4 (GND)
- net MISO: now also R6.1, U4.2 (DO(IO1))
- net MOSI: now also R5.1, U4.5 (DI(IO0))
- net SCK: now also U4.6 (CLK)
- net at J1.2 (Pin_2), J8.2 (Pin_2): now also F3.1, JP3.1 (A); no longer D1.2 (A)
- net at J4.1 (Pin_1), Q2.2: now also R11.1; no longer U2.8
- net at J4.2 (Pin_2): now also F2.1; no longer J10.2 (Pin_2)
- net at J11.1 (DAT2): now also R3.1
- net at J11.8 (DAT1): now also R7.1
- net at J2.1 (Pin_1), Q1.2: now also R10.1; no longer U2.6
- net at J2.2 (Pin_2): now also F1.1; no longer J9.2 (Pin_2)
- net TX: now reaches A1.1 (D1/TX)
- net TX: now also J12.2 (Pin_2)
- net SPI_CS_FLASH: now reaches A1.13 (D10)
- net SPI_CS_FLASH: now also R9.2, U4.1 (~{CS})
- net RX: now reaches A1.2 (D0/RX)
- net RX: now also J12.1 (Pin_1)
- net Buzzer: no longer names the net of BZ1.1 (-)
- net Buzzer: now also U3.3; no longer A1.7 (D4)
- new net: F1.2, J9.2 (Pin_2), JP1.1 (A)
- new net: D3.2 (A), R10.2
- new net: C2.1, J11.4 (VDD)
- new net: D4.2 (A), R8.1
- new net: D1.2 (A), F3.2
- new net: F2.2, J10.2 (Pin_2), JP2.1 (A)
- new net: D2.2 (A), R11.2
- new net BuzzerPin: A1.7 (D4), U3.1
Other:
- moved on the sheet: C1, D1, J1, Q1, Q2, R1, R2, U2A, U2B
